File: KiCAD/GeoRAM/OpenC64Cart.kicad_sch (KiCad schematic)
At the start: 10 parts, among them U1 74HC04, U2 74LS08, U3 74LS00, U4 74LS573, U5 74LS573, U6 74HC245, U7 C64-Exp-Port

Commit message: Fixed some problems on the PCB that prevent the correct parsing on PCBWay
Other:
- company: SukkoPera -> Home Computer Group
- title: OpenC64Cart: C64 8K Lo/Hi-Rom Cartridge -> GEORAM Clone
Changed lines of the file:
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@@
   (paper "A3")
   (title_block
-    (title "OpenC64Cart: C64 8K Lo/Hi-Rom Cartridge")
-    (date "2018-01-04")
-    (rev "2")
-    (company "SukkoPera")
-    (comment 1 "Thanks to http://blog.worldofjani.com/?p=879")
+    (title "GEORAM Clone")
+    (date "2023-01-09")
+    (rev "0")
+    (company "Home Computer Group")
   )
   (junction (at 275.082 82.804) (diameter 0) (color 0 0 0 0)

Commit message: Version 2.0, fixed several issues with the original design
Parts:
- added C1, C2, C3, C4, C5, C8: 100n, Capacitor_THT:C_Disc_D3.0mm_W1.6mm_P2.50mm, symbol OpenC64Cart-rescue:C
- C7: renamed from C1; footprint OpenC64Cart:C_0805+THT -> Capacitor_THT:C_Disc_D3.0mm_W1.6mm_P2.50mm
- U1, U2, U3: footprint Package_DIP:DIP-14_W10.16mm_LongPads -> Package_DIP:DIP-14_W7.62mm
- U1, U2, U3: footprint (none) -> Package_DIP:DIP-14_W7.62mm
- U4, U6: footprint Package_DIP:DIP-20_W7.62mm_LongPads -> Package_DIP:DIP-20_W7.62mm
- U5: footprint Package_DIP:DIP-20_W7.62mm_LongPads -> Package_DIP:DIP-20_W7.62mm; now left out of the parts list
Connections:
- net +5V: now also C1.2, C2.2, C3.2, C4.2, C5.2, C8.2
- net GND: now also C1.1, C2.1, C3.1, C4.1, C5.1, C8.1
Other:
- moved on the sheet: U3E
